File: nonorf.kicad_sch (KiCad schematic)
At the start: 77 parts, among them J1 USB_C_Receptacle, Q1 Si1308EDL, U1 nRF52833/nRF52840-QIxx, U2 NPM1300-QEAA-R7, U3 BME280, Y1 32MHz, Y2 32.768kHz

Commit message: finalize design more or less
Parts:
- removed BZ1: Buzzer, symbol Device:Buzzer
- added H1, H2, H3: MountingHole_Pad, MountingHole:MountingHole_2.1mm, symbol Mechanical:MountingHole_Pad
- added J2: Conn_01x03, Connector_PinHeader_2.54mm:PinHeader_1x03_P2.54mm_Vertical, symbol Connector_Generic:Conn_01x03
- added TP3: TestPoint, TestPoint:TestPoint_Pad_D1.5mm, symbol Connector:TestPoint
- added TP4, TP5, TP6, TP7, TP8: TestPoint, TestPoint:TestPoint_Pad_D1.0mm, symbol Connector:TestPoint
- C15: footprint Capacitor_SMD:C_0402_1005Metric -> Capacitor_SMD:C_0603_1608Metric
- D1, D2, D3, U2, U3: now not fitted
- L1: value 4.7nH -> 3.9nH
- R1, R2: now not fitted; now left out of the parts list
- R3: value 250k -> 470k
- R8: footprint Resistor_SMD:R_0402_1005Metric -> Resistor_SMD:R_0603_1608Metric
- TP1, TP2: footprint TestPoint:TestPoint_Pad_D1.5mm -> TestPoint:TestPoint_Pad_D1.0mm
- U1: value nRF52833/nRF52840-QIxx -> nRF52840-QIAA-R; MPN NRF52833-QIAA-R -> NRF52840-QIAA-R
- Y2: footprint Crystal:Crystal_SMD_2012-2Pin_2.0x1.2mm -> Crystal:Crystal_SMD_3215-2Pin_3.2x1.5mm
Connections:
- net +1V8: now also TP5.1
- net +3V3: now also TP4.1
- net DISP_BUSY: now also U1.A8 (P0.31/AIN7)
- net DISP_CS: now also U1.A14 (P0.19)
- net DISP_D/C: now also U1.A12 (P0.02/AIN0)
- net DISP_MOSI: now also U1.A20 (P0.25)
- net DISP_RES: now also U1.A10 (P0.29/AIN5)
- net DISP_SCLK: now also U1.A16 (P1.05)
- net GND: now also FPC1.26, H1.1, H2.1, H3.1, J2.3 (Pin_3), TP3.1
- net LDO2_OUT: now also TP6.1
- net RESE: now also U1.G1 (P0.26)
- net VSH: now also TP7.1
- net VSL: now also TP8.1
- net Rot_ChA: now reaches U1.AD20 (P0.24)
- net Rot_ChA: now also J2.1 (Pin_1)
- net Rot_ChB: now reaches U1.AD22 (P1.00)
- net Rot_ChB: now also J2.2 (Pin_2)
- no-connect marks 34 -> 28
Other:
- note added: ">250k = 3.3v on VOUT2 (standard reference 150k)"
- note added: "Check if handsolder is possible"
- note added: "jumpers for 0402 resistors in case the RF gods smite us"
- note removed: "250k = 3.3v on VOUT2 (standard reference 150k)"
- note removed: "TODO: CONNECT PMIC I2C TO NRF52840 (SCHEMATIC AND PCB)"
- note removed: "jumpers for 0402 resistors in case impedance fuckery hits us"
- moved on the sheet: C33, C34, C35, C36, C37, C38, C39, C40, C41, C42, C43, D4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

Commit message: final updates to board layout
Parts:
- added TP9: TestPoint, TestPoint:TestPoint_Pad_D1.0mm, symbol Connector:TestPoint
- D4, D5, D6: now not fitted
Connections:
- net DISP_BS: now also U1.J1 (P0.04/AIN2)
- net SW2_RESET: now also TP9.1
Other:
- note added: "Eink"
- note added: "rotary encoder"
- moved on the sheet: C21, C22, C35, C36, C37, C38, C39, C40, C41, C42, C43, FPC1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
