File: nonorf.kicad_pcb (KiCad board)
At the start: 2 copper layers, 38 x 38 mm, 76 parts, among them J1 USB_C_Receptacle, J3 Conn_01x02, Q1 Si1308EDL, U1 nRF52833/nRF52840-QIxx, U2 NPM1300-QEAA-R7, U3 BME280, Y1 32MHz, Y2 32.768kHz

Commit message: finalize design more or less
Parts:
- removed R1, R2: 4.7k, Resistor_SMD:R_0402_1005Metric
- added G***: LOGO, LOGO, F.Cu at (46.8, 18.6)
- added H1: MountingHole_Pad, MountingHole:MountingHole_2.1mm, F.Cu at (15.0, 14.9)
- added H2: MountingHole_Pad, MountingHole:MountingHole_2.1mm, F.Cu at (15.0, 47.0)
- added H3: MountingHole_Pad, MountingHole:MountingHole_2.1mm, F.Cu at (47.0, 47.0)
- added J2: Conn_01x03, Connector_PinHeader_2.54mm:PinHeader_1x03_P2.54mm_Vertical, F.Cu at (47.7, 27.0)
- added TP3: TestPoint, TestPoint:TestPoint_Pad_D1.5mm, F.Cu at (33.4, 17.6)
- added TP4: TestPoint, TestPoint:TestPoint_Pad_D1.0mm, F.Cu at (48.5, 34.4)
- added TP5: TestPoint, TestPoint:TestPoint_Pad_D1.0mm, F.Cu at (45.5, 44.5)
- added TP6: TestPoint, TestPoint:TestPoint_Pad_D1.0mm, F.Cu at (40.1, 44.9)
- added TP7: TestPoint, TestPoint:TestPoint_Pad_D1.0mm, B.Cu at (24.6, 47.2)
- added TP8: TestPoint, TestPoint:TestPoint_Pad_D1.0mm, B.Cu at (22.7, 47.1)
- C15: footprint Capacitor_SMD:C_0402_1005Metric -> Capacitor_SMD:C_0603_1608Metric
- L1: value 4.7nH -> 3.9nH
- R3: value 250k -> 470k
- R8: footprint Resistor_SMD:R_0402_1005Metric -> Resistor_SMD:R_0603_1608Metric
- TP1, TP2: footprint TestPoint:TestPoint_Pad_D1.5mm -> TestPoint:TestPoint_Pad_D1.0mm
- U1: value nRF52833/nRF52840-QIxx -> nRF52840-QIAA-R
- Y2: footprint Crystal:Crystal_SMD_2012-2Pin_2.0x1.2mm -> Crystal:Crystal_SMD_3215-2Pin_3.2x1.5mm
- moved C17 145.5 mm to (28.7, 34.9)
- moved C16 143.8 mm to (28.7, 32.8), turned to -90 degrees
- moved R8 143.8 mm to (21.2, 38.9)
- moved Y2 143.1 mm to (30.4, 33.9)
- moved Q1 142.7 mm to (21.5, 41.0)
- moved R9 142.0 mm to (23.9, 42.3), turned to -45 degrees
- moved J3 141.5 mm to (31.3, 39.0), turned to 180 degrees
- moved D4 141.2 mm to (17.1, 41.6)
- moved D5 139.9 mm to (14.9, 41.6), turned to -90 degrees
- moved C24 139.5 mm to (44.4, 41.4)
- moved C25 139.5 mm to (44.4, 38.2)
- moved C26 139.5 mm to (47.2, 43.3)
- moved C29 139.5 mm to (33.7, 41.2)
- moved R3 139.5 mm to (37.9, 35.4)
- moved R4 139.5 mm to (37.0, 36.2)
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Connections:
- FPC1 pad 26: unconnected-(FPC1-Pad26) -> GND
- U1 pad A10: unconnected-(U1-P0.29/AIN5-PadA10) -> /DISP_RES
- U1 pad A12: unconnected-(U1-P0.02/AIN0-PadA12) -> /DISP_D/C
- U1 pad A14: unconnected-(U1-P0.19-PadA14) -> /DISP_CS
- U1 pad A16: unconnected-(U1-P1.05-PadA16) -> /DISP_SCLK
- U1 pad A20: unconnected-(U1-P0.25-PadA20) -> /DISP_MOSI
- U1 pad A8: unconnected-(U1-P0.31/AIN7-PadA8) -> /DISP_BUSY
- U1 pad AD20: unconnected-(U1-P0.24-PadAD20) -> /Rot_ChA
- U1 pad AD22: unconnected-(U1-P1.00-PadAD22) -> /Rot_ChB
- U1 pad G1: unconnected-(U1-P0.26-PadG1) -> /RESE
Routing:
- net /DISP_MOSI: track 0.00 -> 28.2 mm, vias 0 -> 1
- net /DISP_SCLK: track 0.00 -> 27.8 mm, vias 0 -> 1
- net /DISP_CS: track 0.00 -> 27.6 mm, vias 0 -> 1
- net /DISP_BUSY: track 0.00 -> 25.0 mm, vias 0 -> 1
- net /RESE: track 0.00 -> 25.0 mm, vias 0 -> 1
- net /DISP_D/C: track 0.00 -> 25.0 mm, vias 0 -> 1
- net /DISP_RES: track 0.00 -> 25.0 mm, vias 0 -> 1
- net VSYS: track 2.98 -> 21.0 mm, vias 3 -> 4
- net /GDR: track 3.19 -> 15.4 mm
- net /Rot_ChA: track 0.00 -> 6.73 mm
- net /Rot_ChB: track 0.00 -> 6.07 mm
- net VBUSOUT: track 31.4 -> 25.9 mm
- net Net-(D5-A): track 4.46 -> 9.82 mm
- net Net-(U1-P0.01/XL2): track 7.31 -> 12.6 mm
- net Net-(U1-P0.00/XL1): track 9.06 -> 13.2 mm
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- added copper zone on F.Cu, net +1V8
Other:
- board text added: "CLK"
- board text added: "DIO"
- board text added: "ch_a"
- board text added: "ch_b"

Commit message: final updates to board layout
Parts:
- added G***: LOGO, LOGO, F.Cu at (14.4, 23.6)
- added TP9: TestPoint, TestPoint:TestPoint_Pad_D1.0mm, F.Cu at (45.6, 27.0)
- moved R9 3.66 mm to (23.2, 38.7), turned to 90 degrees
- moved G*** 1.13 mm to (45.9, 19.2)
- moved C17 0.25 mm to (28.7, 34.7)
Connections:
- U1 pad J1: unconnected-(U1-P0.04/AIN2-PadJ1) -> /DISP_BS
Routing:
- net /DISP_BS: track 0.00 -> 25.1 mm, vias 0 -> 1
- net /SW2_RESET: track 0.00 -> 4.45 mm
- net /GDR: track 15.4 -> 16.9 mm
- net /RESE: track 25.0 -> 24.5 mm
- net /DISP_D/C: track 25.0 -> 25.6 mm
- net GND: track 12.8 -> 12.6 mm, vias 122 -> 126
- net (no net): vias 3 -> 0
Other:
- board text added: "Ch_A"
- board text added: "Ch_B"
- board text added: "Clk"
- board text added: "Dio"
- board text added: "Gnd"
- board text added: "VBat"
- board text added: "With love, by Ambraglow"
- board text removed: "CLK"
- board text removed: "DIO"
- board text removed: "ch_a"
- board text removed: "ch_b"

Commit message: silkscreen update
Parts:
- moved G*** 6.44 mm to (20.6, 22.0)
